File: OldStyleDigitalClock_time.kicad_sch (KiCad schematic)
At the start: 13 parts, among them U12 CD4060BE, U13 CD4017BE, U14 CD4017BE, U15 CD4017BE, Y1 HC49 XTAL (32768 Hz)

Commit message: Changed footprints for easy to find parts
Parts:
- U12, U13, U14, U15: footprint Package_SO:SOIC-16W_5.3x10.2mm_P1.27mm -> Package_SO:SOP-16_3.9x9.9mm_P1.27mm
Changed lines of the file:
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@@
 			)
 		)
-		(property "Footprint" "Package_SO:SOIC-16W_5.3x10.2mm_P1.27mm"
+		(property "Footprint" "Package_SO:SOP-16_3.9x9.9mm_P1.27mm"
 			(at 83.82 125.73 0)
 			(effects
@@
 			)
 		)
-		(property "Footprint" "Package_SO:SOIC-16W_5.3x10.2mm_P1.27mm"
+		(property "Footprint" "Package_SO:SOP-16_3.9x9.9mm_P1.27mm"
 			(at 95.25 49.53 0)
 			(effects
@@
 			)
 		)
-		(property "Footprint" "Package_SO:SOIC-16W_5.3x10.2mm_P1.27mm"
+		(property "Footprint" "Package_SO:SOP-16_3.9x9.9mm_P1.27mm"
 			(at 158.75 125.73 0)
 			(effects
@@
 			)
 		)
-		(property "Footprint" "Package_SO:SOIC-16W_5.3x10.2mm_P1.27mm"
+		(property "Footprint" "Package_SO:SOP-16_3.9x9.9mm_P1.27mm"
 			(at 232.41 125.73 0)
 			(effects
