File: OldStyleDigitalClock_time.kicad_sch (KiCad schematic)
At the start: 13 parts, among them U12 CD4060BE, U13 CD4017BE, U14 CD4017BE, U15 CD4017BE, Y1 HC49 XTAL (32768 Hz)

Commit message: Checked all IC against database and updated exact value and footprints
Parts:
- U12: value CD4060BE -> CD4060BM; footprint Package_SO:SOIC-16W_5.3x10.2mm_P1.27mm -> Package_SO:SOIC-16_3.9x9.9mm_P1.27mm
- U13, U14, U15: value CD4017BE -> CD4017BM; footprint Package_SO:SOIC-16W_5.3x10.2mm_P1.27mm -> Package_SO:SOIC-16_3.9x9.9mm_P1.27mm
Changed lines of the file:
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@@
 			)
 		)
-		(property "Value" "CD4017BE"
+		(property "Value" "CD4017BM"
 			(at 83.82 100.33 0)
 			(effects
@@
 			)
 		)
-		(property "Footprint" "Package_SO:SOIC-16W_5.3x10.2mm_P1.27mm"
+		(property "Footprint" "Package_SO:SOIC-16_3.9x9.9mm_P1.27mm"
 			(at 83.82 125.73 0)
 			(effects
@@
 			)
 		)
-		(property "Datasheet" ""
+		(property "Datasheet" "https://www.ti.com/lit/ds/symlink/cd4017b.pdf"
 			(at 83.82 125.73 0)
 			(effects
@@
 			)
 		)
-		(property "Value" "CD4060BE"
+		(property "Value" "CD4060BM"
 			(at 95.25 26.67 0)
 			(effects
@@
 			)
 		)
-		(property "Footprint" "Package_SO:SOIC-16W_5.3x10.2mm_P1.27mm"
-			(at 95.25 49.53 0)
-			(effects
-				(font
-					(size 1.27 1.27)
-				)
-				(justify bottom)
-				(hide yes)
-			)
-		)
-		(property "Datasheet" ""
+		(property "Footprint" "Package_SO:SOIC-16_3.9x9.9mm_P1.27mm"
+			(at 95.25 49.53 0)
+			(effects
+				(font
+					(size 1.27 1.27)
+				)
+				(justify bottom)
+				(hide yes)
+			)
+		)
+		(property "Datasheet" "https://www.ti.com/lit/ds/symlink/cd4060b.pdf"
 			(at 95.25 49.53 0)
 			(effects
@@
 			)
 		)
-		(property "Value" "CD4017BE"
+		(property "Value" "CD4017BM"
 			(at 158.75 100.33 0)
 			(effects
@@
 			)
 		)
-		(property "Footprint" "Package_SO:SOIC-16W_5.3x10.2mm_P1.27mm"
+		(property "Footprint" "Package_SO:SOIC-16_3.9x9.9mm_P1.27mm"
 			(at 158.75 125.73 0)
 			(effects
@@
 			)
 		)
-		(property "Datasheet" ""
+		(property "Datasheet" "https://www.ti.com/lit/ds/symlink/cd4017b.pdf"
 			(at 158.75 125.73 0)
 			(effects
@@
 			)
 		)
-		(property "Value" "CD4017BE"
+		(property "Value" "CD4017BM"
 			(at 232.41 100.33 0)
 			(effects
@@
 			)
 		)
-		(property "Footprint" "Package_SO:SOIC-16W_5.3x10.2mm_P1.27mm"
+		(property "Footprint" "Package_SO:SOIC-16_3.9x9.9mm_P1.27mm"
 			(at 232.41 125.73 0)
 			(effects
@@
 			)
 		)
-		(property "Datasheet" ""
+		(property "Datasheet" "https://www.ti.com/lit/ds/symlink/cd4017b.pdf"
 			(at 232.41 125.73 0)
 			(effects
