File: OldStyleDigitalClock.kicad_sch (KiCad schematic)
At the start: 52 parts, among them SW1 Set minutes, SW2 Set hours, U1 D168K, U10 D168K, U11 CD4026BE, U12 D168K, U13 CD4026BE, U15 4071, U2 CD4026BE, U4 D168K, U5 CD4026BE, U9 4073

Commit message: Partial commit: Moved to SMD footprints
Parts:
- C1: footprint Capacitor_THT:C_Disc_D5.1mm_W3.2mm_P5.00mm -> Capacitor_SMD:C_1206_3216Metric
- C2: renamed from C3; footprint Capacitor_THT:C_Disc_D5.1mm_W3.2mm_P5.00mm -> Capacitor_SMD:C_1206_3216Metric
- C3: renamed from C7; footprint Capacitor_THT:C_Disc_D5.1mm_W3.2mm_P5.00mm -> Capacitor_SMD:C_1206_3216Metric
- C4: renamed from C13; footprint Capacitor_THT:C_Disc_D5.1mm_W3.2mm_P5.00mm -> Capacitor_SMD:C_1206_3216Metric
- C5: renamed from C12; footprint Capacitor_THT:C_Disc_D5.1mm_W3.2mm_P5.00mm -> Capacitor_SMD:C_1206_3216Metric
- C6: renamed from C19; footprint Capacitor_THT:C_Disc_D5.1mm_W3.2mm_P5.00mm -> Capacitor_SMD:C_1206_3216Metric
- C7: renamed from C11; footprint Capacitor_THT:C_Disc_D5.1mm_W3.2mm_P5.00mm -> Capacitor_SMD:C_1206_3216Metric
- C8: renamed from C15; footprint Capacitor_THT:C_Disc_D5.1mm_W3.2mm_P5.00mm -> Capacitor_SMD:C_1206_3216Metric
- R1, R2, R7, R8, R9: footprint Resistor_THT:R_Axial_DIN0204_L3.6mm_D1.6mm_P7.62mm_Horizontal -> Resistor_SMD:R_1206_3216Metric
- R10: renamed from R11; footprint Resistor_THT:R_Axial_DIN0204_L3.6mm_D1.6mm_P7.62mm_Horizontal -> Resistor_SMD:R_1206_3216Metric
- R11: renamed from R12; footprint Resistor_THT:R_Axial_DIN0204_L3.6mm_D1.6mm_P7.62mm_Horizontal -> Resistor_SMD:R_1206_3216Metric
- R12: renamed from R13; footprint Resistor_THT:R_Axial_DIN0204_L3.6mm_D1.6mm_P7.62mm_Horizontal -> Resistor_SMD:R_1206_3216Metric
- R13: renamed from R14; footprint Resistor_THT:R_Axial_DIN0204_L3.6mm_D1.6mm_P7.62mm_Horizontal -> Resistor_SMD:R_1206_3216Metric
- R14: renamed from R15; footprint Resistor_THT:R_Axial_DIN0204_L3.6mm_D1.6mm_P7.62mm_Horizontal -> Resistor_SMD:R_1206_3216Metric
- R15: renamed from R16; footprint Resistor_THT:R_Axial_DIN0204_L3.6mm_D1.6mm_P7.62mm_Horizontal -> Resistor_SMD:R_1206_3216Metric
- R16: renamed from R17; footprint Resistor_THT:R_Axial_DIN0204_L3.6mm_D1.6mm_P7.62mm_Horizontal -> Resistor_SMD:R_1206_3216Metric
- R17: renamed from R19; footprint Resistor_THT:R_Axial_DIN0204_L3.6mm_D1.6mm_P7.62mm_Horizontal -> Resistor_SMD:R_1206_3216Metric
- R18: renamed from R23; footprint Resistor_THT:R_Axial_DIN0204_L3.6mm_D1.6mm_P7.62mm_Horizontal -> Resistor_SMD:R_1206_3216Metric
- R19: renamed from R20; footprint Resistor_THT:R_Axial_DIN0204_L3.6mm_D1.6mm_P7.62mm_Horizontal -> Resistor_SMD:R_1206_3216Metric
- R20: renamed from R21; footprint Resistor_THT:R_Axial_DIN0204_L3.6mm_D1.6mm_P7.62mm_Horizontal -> Resistor_SMD:R_1206_3216Metric
- R21: renamed from R22; footprint Resistor_THT:R_Axial_DIN0204_L3.6mm_D1.6mm_P7.62mm_Horizontal -> Resistor_SMD:R_1206_3216Metric
- R22: renamed from R24; footprint Resistor_THT:R_Axial_DIN0204_L3.6mm_D1.6mm_P7.62mm_Horizontal -> Resistor_SMD:R_1206_3216Metric
- R23: renamed from R25; footprint Resistor_THT:R_Axial_DIN0204_L3.6mm_D1.6mm_P7.62mm_Horizontal -> Resistor_SMD:R_1206_3216Metric
- R24: renamed from R26; footprint Resistor_THT:R_Axial_DIN0204_L3.6mm_D1.6mm_P7.62mm_Horizontal -> Resistor_SMD:R_1206_3216Metric
- R25: renamed from R27; footprint Resistor_THT:R_Axial_DIN0204_L3.6mm_D1.6mm_P7.62mm_Horizontal -> Resistor_SMD:R_1206_3216Metric
- R26: renamed from R28; footprint Resistor_THT:R_Axial_DIN0204_L3.6mm_D1.6mm_P7.62mm_Horizontal -> Resistor_SMD:R_1206_3216Metric
- R27: renamed from R29; footprint Resistor_THT:R_Axial_DIN0204_L3.6mm_D1.6mm_P7.62mm_Horizontal -> Resistor_SMD:R_1206_3216Metric
- R28: renamed from R30; footprint Resistor_THT:R_Axial_DIN0204_L3.6mm_D1.6mm_P7.62mm_Horizontal -> Resistor_SMD:R_1206_3216Metric
- R29: renamed from R31; footprint Resistor_THT:R_Axial_DIN0204_L3.6mm_D1.6mm_P7.62mm_Horizontal -> Resistor_SMD:R_1206_3216Metric
- R3: renamed from R4; footprint Resistor_THT:R_Axial_DIN0204_L3.6mm_D1.6mm_P7.62mm_Horizontal -> Resistor_SMD:R_1206_3216Metric
- R30: renamed from R32; footprint Resistor_THT:R_Axial_DIN0204_L3.6mm_D1.6mm_P7.62mm_Horizontal -> Resistor_SMD:R_1206_3216Metric
- R31: renamed from R33; footprint Resistor_THT:R_Axial_DIN0204_L3.6mm_D1.6mm_P7.62mm_Horizontal -> Resistor_SMD:R_1206_3216Metric
- R32: renamed from R34; footprint Resistor_THT:R_Axial_DIN0204_L3.6mm_D1.6mm_P7.62mm_Horizontal -> Resistor_SMD:R_1206_3216Metric
- R4: renamed from R5; footprint Resistor_THT:R_Axial_DIN0204_L3.6mm_D1.6mm_P7.62mm_Horizontal -> Resistor_SMD:R_1206_3216Metric
- R5: renamed from R6; footprint Resistor_THT:R_Axial_DIN0204_L3.6mm_D1.6mm_P7.62mm_Horizontal -> Resistor_SMD:R_1206_3216Metric
- R6: renamed from R3; footprint Resistor_THT:R_Axial_DIN0204_L3.6mm_D1.6mm_P7.62mm_Horizontal -> Resistor_SMD:R_1206_3216Metric
- renumbered U15 to U1, U13 to U10, U1 to U2, U2 to U3, U9 to U6, U10 to U7, U11 to U8, U12 to U9

Commit message: Removed old footprints
Parts:
- U10, U3, U5, U8: footprint CD4026BE:DIP794W45P254L1969H508Q16 -> (none)
- U6: footprint CD4073BE:DIP794W45P254L1969H508Q14 -> (none)
Changed lines of the file:
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@@
 			)
 		)
-		(property "Footprint" "CD4026BE:DIP794W45P254L1969H508Q16"
+		(property "Footprint" ""
 			(at 201.93 184.15 0)
 			(effects
@@
 			)
 		)
-		(property "Footprint" "CD4073BE:DIP794W45P254L1969H508Q14"
+		(property "Footprint" ""
 			(at 43.18 133.35 0)
 			(effects
@@
 			)
 		)
-		(property "Footprint" "CD4073BE:DIP794W45P254L1969H508Q14"
+		(property "Footprint" ""
 			(at 43.18 222.25 0)
 			(effects
@@
 			)
 		)
-		(property "Footprint" "CD4026BE:DIP794W45P254L1969H508Q16"
+		(property "Footprint" ""
 			(at 279.4 46.99 0)
 			(effects
@@
 			)
 		)
-		(property "Footprint" "CD4026BE:DIP794W45P254L1969H508Q16"
+		(property "Footprint" ""
 			(at 280.67 109.22 0)
 			(effects
@@
 			)
 		)
-		(property "Footprint" "CD4026BE:DIP794W45P254L1969H508Q16"
+		(property "Footprint" ""
 			(at 203.2 246.38 0)
 			(effects
@@
 			)
 		)
-		(property "Footprint" "CD4073BE:DIP794W45P254L1969H508Q14"
+		(property "Footprint" ""
 			(at 203.2 278.13 0)
 			(effects
@@
 			)
 		)
-		(property "Footprint" "CD4073BE:DIP794W45P254L1969H508Q14"
+		(property "Footprint" ""
 			(at 281.94 140.97 0)
 			(effects

Commit message: Assigned footprints: first draft
Parts:
- U1, U6: footprint (none) -> Package_SO:SO-14_5.3x10.2mm_P1.27mm
- U10, U3, U5, U8: footprint (none) -> Package_SO:SOIC-16W_5.3x10.2mm_P1.27mm
Changed lines of the file:
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@@
 			)
 		)
-		(property "Footprint" ""
+		(property "Footprint" "Package_SO:SO-14_5.3x10.2mm_P1.27mm"
 			(at 134.62 250.19 0)
 			(effects
@@
 			)
 		)
-		(property "Footprint" ""
+		(property "Footprint" "Package_SO:SOIC-16W_5.3x10.2mm_P1.27mm"
 			(at 201.93 184.15 0)
 			(effects
@@
 			)
 		)
-		(property "Footprint" ""
+		(property "Footprint" "Package_SO:SO-14_5.3x10.2mm_P1.27mm"
 			(at 210.82 34.29 0)
 			(effects
@@
 			)
 		)
-		(property "Footprint" ""
+		(property "Footprint" "Package_SO:SO-14_5.3x10.2mm_P1.27mm"
 			(at 43.18 170.18 0)
 			(effects
@@
 			)
 		)
-		(property "Footprint" ""
+		(property "Footprint" "Package_SO:SO-14_5.3x10.2mm_P1.27mm"
 			(at 43.18 133.35 0)
 			(effects
@@
 			)
 		)
-		(property "Footprint" ""
+		(property "Footprint" "Package_SO:SO-14_5.3x10.2mm_P1.27mm"
 			(at 43.18 222.25 0)
 			(effects
@@
 			)
 		)
-		(property "Footprint" ""
+		(property "Footprint" "Package_SO:SO-14_5.3x10.2mm_P1.27mm"
 			(at 154.94 147.32 0)
 			(effects
@@
 			)
 		)
-		(property "Footprint" ""
+		(property "Footprint" "Package_SO:SOIC-16W_5.3x10.2mm_P1.27mm"
 			(at 279.4 46.99 0)
 			(effects
@@
 			)
 		)
-		(property "Footprint" ""
+		(property "Footprint" "Package_SO:SOIC-16W_5.3x10.2mm_P1.27mm"
 			(at 280.67 109.22 0)
 			(effects
@@
 			)
 		)
-		(property "Footprint" ""
+		(property "Footprint" "Package_SO:SOIC-16W_5.3x10.2mm_P1.27mm"
 			(at 203.2 246.38 0)
 			(effects
@@
 			)
 		)
-		(property "Footprint" ""
+		(property "Footprint" "Package_SO:SO-14_5.3x10.2mm_P1.27mm"
 			(at 203.2 278.13 0)
 			(effects
@@
 			)
 		)
-		(property "Footprint" ""
+		(property "Footprint" "Package_SO:SO-14_5.3x10.2mm_P1.27mm"
 			(at 281.94 140.97 0)
 			(effects
@@
 			)
 		)
-		(property "Footprint" ""
+		(property "Footprint" "Package_SO:SO-14_5.3x10.2mm_P1.27mm"
 			(at 226.06 120.65 0)
 			(effects

Commit message: Tracks 1
Connections:
- no-connect marks 1 -> 5
Changed lines of the file:
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@@
+	)
+	(no_connect
+		(at 378.46 52.07)
+	)
+	(no_connect
+		(at 378.46 189.23)
+	)
+	(no_connect
+		(at 378.46 236.22)
 	)
 	(no_connect
 		(at 50.8 133.35)
 	)
+	(no_connect
+		(at 378.46 114.3)
+	)
 	(wire

Commit message: Moved USB receptacles, minor changes. Marked no connect pins.
Connections:
- no-connect marks 5 -> 12
Changed lines of the file:
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@@
 	(title_block
 		(title "Old style digital clock")
-		(date "2025-10-13")
+		(date "2025-11-08")
 		(rev "1")
 		(company "Pasquale Lafiosca")
@@
 	)
 	(no_connect
+		(at 238.76 246.38)
+	)
+	(no_connect
 		(at 378.46 52.07)
+	)
+	(no_connect
+		(at 316.23 104.14)
+	)
+	(no_connect
+		(at 238.76 241.3)
+	)
+	(no_connect
+		(at 238.76 256.54)
+	)
+	(no_connect
+		(at 237.49 194.31)
 	)
 	(no_connect
@@
 	)
 	(no_connect
+		(at 316.23 119.38)
+	)
+	(no_connect
 		(at 378.46 114.3)
 	)
+	(no_connect
+		(at 314.96 57.15)
+	)
 	(wire

Commit message: Reviewed LED limiting resistors to stay within specs
Parts:
- R10, R11, R12, R13, R14, R15, R16, R19, R2, R20, R21, R22, R23, R24, R25, R26, R27, R28, R29, R3, R30, R31, R32, R4, R5, R7, R8, R9: value 2.2 kΩ -> 4.7 kΩ
Other:
- note removed: "Value of resistors may need to be adjusted according to the chosen 7 segment LEDs."
Changed lines of the file:
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@@
 		(company "Pasquale Lafiosca")
 	)
-	(text "Value of resistors may need\nto be adjusted according to\nthe chosen 7 segment LEDs."
-		(exclude_from_sim no)
-		(at 345.44 30.48 0)
-		(effects
-			(font
-				(size 1.27 1.27)
-			)
-			(justify left bottom)
-		)
-	)
 	(junction
 		(at 35.56 133.35)
@@
 			)
 		)
-		(property "Value" "2.2 kΩ"
+		(property "Value" "4.7 kΩ"
 			(at 355.6 181.61 90)
 			(effects
@@
 			)
 		)
-		(property "Value" "2.2 kΩ"
+		(property "Value" "4.7 kΩ"
 			(at 325.12 31.75 90)
 			(effects
@@
 			)
 		)
-		(property "Value" "2.2 kΩ"
+		(property "Value" "4.7 kΩ"
 			(at 363.22 184.15 90)
 			(effects
@@
 			)
 		)
-		(property "Value" "2.2 kΩ"
+		(property "Value" "4.7 kΩ"
 			(at 337.82 36.83 90)
 			(effects
@@
 			)
 		)
-		(property "Value" "2.2 kΩ"
+		(property "Value" "4.7 kΩ"
 			(at 344.17 101.6 90)
 			(effects
@@
 			)
 		)
-		(property "Value" "2.2 kΩ"
+		(property "Value" "4.7 kΩ"
 			(at 340.36 176.53 90)
 			(effects
@@
 			)
 		)
-		(property "Value" "2.2 kΩ"
+		(property "Value" "4.7 kΩ"
 			(at 317.5 168.91 90)
 			(effects
@@
 			)
 		)
-		(property "Value" "2.2 kΩ"
+		(property "Value" "4.7 kΩ"
 			(at 364.49 46.99 90)
 			(effects
@@
 			)
 		)
-		(property "Value" "2.2 kΩ"
+		(property "Value" "4.7 kΩ"
 			(at 356.87 106.68 90)
 			(effects
@@
 			)
 		)
-		(property "Value" "2.2 kΩ"
+		(property "Value" "4.7 kΩ"
 			(at 358.14 44.45 90)
 			(effects
@@
 			)
 		)
-		(property "Value" "2.2 kΩ"
+		(property "Value" "4.7 kΩ"
 			(at 350.52 104.14 90)
 			(effects
@@
 			)
 		)
-		(property "Value" "2.2 kΩ"
+		(property "Value" "4.7 kΩ"
 			(at 320.04 215.9 90)
 			(effects
@@
 			)
 		)
-		(property "Value" "2.2 kΩ"
+		(property "Value" "4.7 kΩ"
 			(at 331.47 96.52 90)
 			(effects
@@
 			)
 		)
-		(property "Value" "2.2 kΩ"
+		(property "Value" "4.7 kΩ"
 			(at 325.12 171.45 90)
 			(effects
@@
 			)
 		)
-		(property "Value" "2.2 kΩ"
+		(property "Value" "4.7 kΩ"
 			(at 340.36 223.52 90)
 			(effects
@@
 			)
 		)
-		(property "Value" "2.2 kΩ"
+		(property "Value" "4.7 kΩ"
 			(at 363.22 231.14 90)
 			(effects
@@
 			)
 		)
-		(property "Value" "2.2 kΩ"
+		(property "Value" "4.7 kΩ"
 			(at 332.74 173.99 90)
 			(effects
@@
 			)
 		)
-		(property "Value" "2.2 kΩ"
+		(property "Value" "4.7 kΩ"
 			(at 355.6 228.6 90)
 			(effects
@@
 			)
 		)
-		(property "Value" "2.2 kΩ"
+		(property "Value" "4.7 kΩ"
 			(at 331.47 34.29 90)
 			(effects
@@
 			)
 		)
-		(property "Value" "2.2 kΩ"
+		(property "Value" "4.7 kΩ"
 			(at 337.82 99.06 90)
 			(effects
@@
 			)
 		)
-		(property "Value" "2.2 kΩ"
+		(property "Value" "4.7 kΩ"
 			(at 344.17 39.37 90)
 			(effects
@@
 			)
 		)
-		(property "Value" "2.2 kΩ"
+		(property "Value" "4.7 kΩ"
 			(at 326.39 218.44 90)
 			(effects
@@
 			)
 		)
-		(property "Value" "2.2 kΩ"
+		(property "Value" "4.7 kΩ"
 			(at 347.98 226.06 90)
 			(effects
@@
 			)
 		)
-		(property "Value" "2.2 kΩ"
+		(property "Value" "4.7 kΩ"
 			(at 363.22 109.22 90)
 			(effects
@@
 			)
 		)
-		(property "Value" "2.2 kΩ"
+		(property "Value" "4.7 kΩ"
 			(at 325.12 93.98 90)
 			(effects
@@
 			)
 		)
-		(property "Value" "2.2 kΩ"
+		(property "Value" "4.7 kΩ"
 			(at 350.52 41.91 90)
 			(effects
@@
 			)
 		)
-		(property "Value" "2.2 kΩ"
+		(property "Value" "4.7 kΩ"
 			(at 332.74 220.98 90)
 			(effects
@@
 			)
 		)
-		(property "Value" "2.2 kΩ"
+		(property "Value" "4.7 kΩ"
 			(at 347.98 179.07 90)
 			(effects

Commit message: Checked all IC against database and updated exact value and footprints
Parts:
- U1: value 4071 -> CD4071BM; footprint Package_SO:SO-14_5.3x10.2mm_P1.27mm -> Package_SO:SOIC-14_3.9x8.7mm_P1.27mm
- U10, U3, U5, U8: value CD4026BE -> CD4026BNSR
- U6: value 4073 -> CD4073BM; footprint Package_SO:SO-14_5.3x10.2mm_P1.27mm -> Package_SO:SOIC-14_3.9x8.7mm_P1.27mm
Changed lines of the file:
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@@
 			)
 		)
-		(property "Value" "4071"
+		(property "Value" "CD4071BM"
 			(at 134.62 243.84 0)
 			(effects
@@
 			)
 		)
-		(property "Footprint" "Package_SO:SO-14_5.3x10.2mm_P1.27mm"
+		(property "Footprint" "Package_SO:SOIC-14_3.9x8.7mm_P1.27mm"
 			(at 134.62 250.19 0)
 			(effects
@@
 			)
 		)
-		(property "Datasheet" "http://www.intersil.com/content/dam/Intersil/documents/cd40/cd4071bms-72bms-75bms.pdf"
+		(property "Datasheet" "https://www.ti.com/lit/ds/symlink/cd4071b.pdf"
 			(at 134.62 250.19 0)
 			(effects
@@
 			)
 		)
-		(property "Value" "CD4026BE"
+		(property "Value" "CD4026BNSR"
 			(at 201.93 161.29 0)
 			(effects
@@
 			)
 		)
-		(property "Datasheet" ""
+		(property "Datasheet" "https://www.ti.com/lit/ds/symlink/cd4026b.pdf?ts=1762977938812"
 			(at 201.93 184.15 0)
 			(effects
@@
 			)
 		)
-		(property "Description" ""
+		(property "Description" "Only SOIC-16W in datasheet"
 			(at 201.93 184.15 0)
 			(effects
@@
 			)
 		)
-		(property "Value" "4071"
+		(property "Value" "CD4071BM"
 			(at 210.82 27.94 0)
 			(effects
@@
 			)
 		)
-		(property "Footprint" "Package_SO:SO-14_5.3x10.2mm_P1.27mm"
+		(property "Footprint" "Package_SO:SOIC-14_3.9x8.7mm_P1.27mm"
 			(at 210.82 34.29 0)
 			(effects
@@
 			)
 		)
-		(property "Datasheet" "http://www.intersil.com/content/dam/Intersil/documents/cd40/cd4071bms-72bms-75bms.pdf"
+		(property "Datasheet" "https://www.ti.com/lit/ds/symlink/cd4071b.pdf"
 			(at 210.82 34.29 0)
 			(effects
@@
 			)
 		)
-		(property "Value" "4071"
+		(property "Value" "CD4071BM"
 			(at 49.53 171.4499 0)
 			(effects
@@
 			)
 		)
-		(property "Footprint" "Package_SO:SO-14_5.3x10.2mm_P1.27mm"
+		(property "Footprint" "Package_SO:SOIC-14_3.9x8.7mm_P1.27mm"
 			(at 43.18 170.18 0)
 			(effects
@@
 			)
 		)
-		(property "Datasheet" "http://www.intersil.com/content/dam/Intersil/documents/cd40/cd4071bms-72bms-75bms.pdf"
+		(property "Datasheet" "https://www.ti.com/lit/ds/symlink/cd4071b.pdf"
 			(at 43.18 170.18 0)
 			(effects
@@
 			)
 		)
-		(property "Value" "4073"
+		(property "Value" "CD4073BM"
 			(at 43.18 127 0)
 			(effects
@@
 			)
 		)
-		(property "Footprint" "Package_SO:SO-14_5.3x10.2mm_P1.27mm"
+		(property "Footprint" "Package_SO:SOIC-14_3.9x8.7mm_P1.27mm"
 			(at 43.18 133.35 0)
 			(effects
@@
 			)
 		)
-		(property "Datasheet" "http://www.intersil.com/content/dam/Intersil/documents/cd40/cd4073bms-81bms-82bms.pdf"
+		(property "Datasheet" "https://www.ti.com/lit/ds/symlink/cd4073b.pdf?ts=1763007214799"
 			(at 43.18 133.35 0)
 			(effects
@@
 			)
 		)
-		(property "Value" "4073"
+		(property "Value" "CD4073BM"
 			(at 49.53 223.5199 0)
 			(effects
@@
 			)
 		)
-		(property "Footprint" "Package_SO:SO-14_5.3x10.2mm_P1.27mm"
+		(property "Footprint" "Package_SO:SOIC-14_3.9x8.7mm_P1.27mm"
 			(at 43.18 222.25 0)
 			(effects
@@
 			)
 		)
-		(property "Datasheet" "http://www.intersil.com/content/dam/Intersil/documents/cd40/cd4073bms-81bms-82bms.pdf"
+		(property "Datasheet" "https://www.ti.com/lit/ds/symlink/cd4073b.pdf?ts=1763007214799"
 			(at 43.18 222.25 0)
 			(effects
@@
 			)
 		)
-		(property "Value" "4071"
+		(property "Value" "CD4071BM"
 			(at 154.94 140.97 0)
 			(effects
@@
 			)
 		)
-		(property "Footprint" "Package_SO:SO-14_5.3x10.2mm_P1.27mm"
+		(property "Footprint" "Package_SO:SOIC-14_3.9x8.7mm_P1.27mm"
 			(at 154.94 147.32 0)
 			(effects
@@
 			)
 		)
-		(property "Datasheet" "http://www.intersil.com/content/dam/Intersil/documents/cd40/cd4071bms-72bms-75bms.pdf"
+		(property "Datasheet" "https://www.ti.com/lit/ds/symlink/cd4071b.pdf"
 			(at 154.94 147.32 0)
 			(effects
@@
 			)
 		)
-		(property "Value" "CD4026BE"
+		(property "Value" "CD4026BNSR"
 			(at 279.4 24.13 0)
 			(effects
@@
 			)
 		)
-		(property "Datasheet" ""
+		(property "Datasheet" "https://www.ti.com/lit/ds/symlink/cd4026b.pdf?ts=1762977938812"
 			(at 279.4 46.99 0)
 			(effects
@@
 			)
 		)
-		(property "Description" ""
+		(property "Description" "Only SOIC-16W in datasheet"
 			(at 279.4 46.99 0)
 			(effects
@@
 			)
 		)
-		(property "Value" "CD4026BE"
+		(property "Value" "CD4026BNSR"
 			(at 280.67 86.36 0)
 			(effects
@@
 			)
 		)
-		(property "Datasheet" ""
+		(property "Datasheet" "https://www.ti.com/lit/ds/symlink/cd4026b.pdf?ts=1762977938812"
 			(at 280.67 109.22 0)
 			(effects
@@
 			)
 		)
-		(property "Description" ""
+		(property "Description" "Only SOIC-16W in datasheet"
 			(at 280.67 109.22 0)
 			(effects
@@
 			)
 		)
-		(property "Value" "CD4026BE"
+		(property "Value" "CD4026BNSR"
 			(at 203.2 223.52 0)
 			(effects
@@
 			)
 		)
-		(property "Datasheet" ""
+		(property "Datasheet" "https://www.ti.com/lit/ds/symlink/cd4026b.pdf?ts=1762977938812"
 			(at 203.2 246.38 0)
 			(effects
@@
 			)
 		)
-		(property "Description" ""
+		(property "Description" "Only SOIC-16W in datasheet"
 			(at 203.2 246.38 0)
 			(effects
@@
 			)
 		)
-		(property "Value" "4073"
+		(property "Value" "CD4073BM"
 			(at 203.2 271.78 0)
 			(effects
@@
 			)
 		)
-		(property "Footprint" "Package_SO:SO-14_5.3x10.2mm_P1.27mm"
+		(property "Footprint" "Package_SO:SOIC-14_3.9x8.7mm_P1.27mm"
 			(at 203.2 278.13 0)
 			(effects
@@
 			)
 		)
-		(property "Datasheet" "http://www.intersil.com/content/dam/Intersil/documents/cd40/cd4073bms-81bms-82bms.pdf"
+		(property "Datasheet" "https://www.ti.com/lit/ds/symlink/cd4073b.pdf?ts=1763007214799"
 			(at 203.2 278.13 0)
 			(effects
@@
 			)
 		)
-		(property "Value" "4073"
+		(property "Value" "CD4073BM"
 			(at 281.94 134.62 0)
 			(effects
@@
 			)
 		)
-		(property "Footprint" "Package_SO:SO-14_5.3x10.2mm_P1.27mm"
+		(property "Footprint" "Package_SO:SOIC-14_3.9x8.7mm_P1.27mm"
 			(at 281.94 140.97 0)
 			(effects
@@
 			)
 		)
-		(property "Datasheet" "http://www.intersil.com/content/dam/Intersil/documents/cd40/cd4073bms-81bms-82bms.pdf"
+		(property "Datasheet" "https://www.ti.com/lit/ds/symlink/cd4073b.pdf?ts=1763007214799"
 			(at 281.94 140.97 0)
 			(effects
@@
 			)
 		)
-		(property "Value" "4071"
+		(property "Value" "CD4071BM"
 			(at 226.06 114.3 0)
 			(effects
@@
 			)
 		)
-		(property "Footprint" "Package_SO:SO-14_5.3x10.2mm_P1.27mm"
+		(property "Footprint" "Package_SO:SOIC-14_3.9x8.7mm_P1.27mm"
 			(at 226.06 120.65 0)
 			(effects
@@
 			)
 		)
-		(property "Datasheet" "http://www.intersil.com/content/dam/Intersil/documents/cd40/cd4071bms-72bms-75bms.pdf"
+		(property "Datasheet" "https://www.ti.com/lit/ds/symlink/cd4071b.pdf"
 			(at 226.06 120.65 0)
 			(effects
